File: kicad/lt15t3/lt15t3.kicad_sch (KiCad schematic)
At the start: 40 parts

Commit message: Finalize PCB design
Parts:
- removed C?: 0.1uF, symbol Device:C_Small
- removed D? (x3): SM4002, Diode_SMD:D_MELF, symbol Diode:SM4002
- removed D? (x4): 15.7V, symbol Device:D_Zener
- added D1, D2: P4SMA18CA, Diode_SMD:D_SMA, symbol Device:D_TVS
- added D5, D6, D9: US1B, Diode_SMD:D_SMA, symbol Diode:US1B
- added J1, J2, J3: Screw_Terminal_01x04, Connector_PinHeader_2.54mm:PinHeader_1x04_P2.54mm_Vertical, symbol Connector:Screw_Terminal_01x04
- C1, C11, C2, C3, C4: renamed from C?; footprint (none) -> Capacitor_SMD:C_0805_2012Metric
- D8: renamed from D?; value 3.3V TVS -> BZY55B3V6 RBG; footprint (none) -> Diode_SMD:D_0805_2012Metric
- F1, F2: renamed from F?; footprint (none) -> Capacitor_THT:C_Disc_D5.1mm_W3.2mm_P5.00mm
- R1, R2, R3, R4, R5, R6, R7, R8: renamed from R?; footprint (none) -> Resistor_SMD:R_0805_2012Metric
- U5: renamed from U?; footprint (none) -> Package_TO_SOT_THT:TO-220-3_Vertical
- U6: renamed from U?; footprint (none) -> Package_SO:SOIC-8W_5.3x5.3mm_P1.27mm
- U6: renamed from U?; footprint (none) -> Package_SO:SOIC-8W_5.3x5.3mm_P1.27mm; MouserNr (none) -> 595-OPA2376AQDRQ1
- gave numbers to parts that had none: 12
Connections:
- net +3V3 is gone; now on net +3.3V: C10.1, U5.3 (OUT)
- net +15V: now also C1.2, D5.1 (K), D9.2 (A); no longer C1.1
- net +3.3V: now also D5.2 (A)
- net -15V: now also D6.1 (K)
- net GND: now also C1.1, D1.1 (A1), D2.1 (A1), J1.2 (Pin_2), J1.4 (Pin_4), J2.2 (Pin_2), J2.4 (Pin_4), J3.2 (Pin_2), J3.4 (Pin_4); no longer C1.2
- net IN1: now also D2.2 (A2), J3.1 (Pin_1)
- net IN2: now also D1.2 (A2), J3.3 (Pin_3)
- net O1: now also J2.1 (Pin_1)
- net O2: now also J2.3 (Pin_3)
- net VCC: now also J1.1 (Pin_1)
- net VSS: now also J1.3 (Pin_3)
- net at C5.1, D3.1 (K), F2.2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: now also D9.1 (K)
- net at C6.2, D4.2 (A), F1.2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: now also D6.2 (A)
